Commit message: rename urdf to RAVEN

File: urdf/urdf/RAVEN.urdf (robot description, URDF)
Before this commit: robot urdf, 4 links, 3 joints
Links:
- link base_link: geometry collision mesh filename=../meshes/base_link.STL; visual mesh filename=../meshes/base_link.STL
- link foreArm_link: geometry collision mesh filename=../meshes/foreArm_link.STL; visual mesh filename=../meshes/foreArm_link.STL
- link shoulder_link: geometry collision mesh filename=../meshes/shoulder_link.STL; visual mesh filename=../meshes/shoulder_link.STL
- link upperArm_link: geometry collision mesh filename=../meshes/upperArm_link.STL; visual mesh filename=../meshes/upperArm_link.STL

Commit message: add forearm link rotation

File: urdf/urdf/RAVEN.urdf (robot description, URDF)
Before this commit: robot urdf, 4 links, 3 joints
Joints:
- joint foreArm_pitch: axis 0 0 0 -> 0 -1 0; limit (none) -> lower=0 upper=3.14 effort=0 velocity=0; type fixed -> revolute

Commit message: rename joint axis

File: urdf/urdf/RAVEN.urdf (robot description, URDF)
Before this commit: robot urdf, 4 links, 3 joints
Joints:
- removed joint shoulder_pitch
- added joint shoulder_yaw: type revolute, parent base_link, child shoulder_link, origin xyz=0 -0.0015 0.1205 rpy=0 0 0, axis 0 0 -1, limit lower=-3.14 upper=3.14 effort=0 velocity=0

Commit message: edit

File: urdf/urdf/RAVEN.urdf (robot description, URDF)
Before this commit: robot urdf, 4 links, 3 joints
Joints:
- joint shoulder_yaw: origin xyz=0 -0.0015 0.1205 rpy=0 0 0 -> xyz=0 0 0.1205 rpy=0 0 0
