Commit message: urdf final version

File: urdf/urdf/RAVEN.urdf (robot description, URDF)
Before this commit: robot RAVEN, 4 links, 3 joints
Links:
- link base_link: mass 0.24946 -> 0.468898
- link foreArm_link: mass 0.16941 -> 0.14102
- link shoulder_link: mass 0.4346 -> 0.598911
- link upperArm_link: mass 0.38582 -> 0.718905
Joints:
- removed joint foreArm_pitch
- removed joint shoulder_yaw
- removed joint upperArm_pitch
- added joint foreArm_Joint: type revolute, parent upperArm_link, child foreArm_link, origin xyz=-0.225 -2.5E-05 -7.5E-05 rpy=0 0 0, axis 0 -1 0, limit lower=0 upper=3.14 effort=0 velocity=0
- added joint shoulder_Joint: type revolute, parent base_link, child shoulder_link, origin xyz=0 0 0.0504 rpy=0 0 0, axis 0 0 1, limit lower=-3.14 upper=3.14 effort=0 velocity=0
- added joint upperArm_Joint: type revolute, parent shoulder_link, child upperArm_link, origin xyz=0 0.027 0.07 rpy=0 0 0, axis 0 1 0, limit lower=0 upper=3.14 effort=0 velocity=0
