Commit message: mass override

File: urdf/urdf/RAVEN_abs.urdf (robot description, URDF)
Before this commit: robot RAVEN, 4 links, 3 joints
Links:
- link base_link: mass 0.24946 -> 0.4535
- link foreArm_link: mass 0.16941 -> 0.1379
- link shoulder_link: mass 0.4346 -> 0.5653
- link upperArm_link: mass 0.38582 -> 0.5692
