Commit message: file organizing

File: legacy/urdf/urdf/RAVEN.urdf (robot description, URDF)
Before this commit: robot RAVEN, 4 links, 3 joints
Links:
- link base_link: mass 0.24552070353348 -> 0.24946
- link foreArm_link: mass 0.210338139477223 -> 0.16941
- link shoulder_link: mass 0.430665397462828 -> 0.4346
- link upperArm_link: mass 0.41988933274855 -> 0.38582
Joints:
- removed joint foreArm_Joint
- removed joint shoulder_Joint
- removed joint upperArm_Joint
- added joint foreArm_pitch: type revolute, parent upperArm_link, child foreArm_link, origin xyz=-0.22125 0 0 rpy=0 0 0, axis 0 -1 0, limit lower=0 upper=3.14 effort=0 velocity=0
- added joint shoulder_yaw: type revolute, parent base_link, child shoulder_link, origin xyz=0 0 0.1205 rpy=0 0 0, axis 0 0 -1, limit lower=-3.14 upper=3.14 effort=0 velocity=0
- added joint upperArm_pitch: type revolute, parent shoulder_link, child upperArm_link, origin xyz=0 0 0 rpy=0 0 0, axis 0 1 0, limit lower=0 upper=3.14 effort=0 velocity=0
